File: hardware/node/_autosave-node.kicad_pcb (KiCad board)
At the start: 2 copper layers, 168.9 x 109.2 mm, 64 parts, among them IC1 MCP73844-840I_MS, IC2 LM2576SX-3.3_NOPB, IC3 LM2585S-12_NOPB, IC4 NEO-M9N-00B, J1 USB4140-GF-0070-C, J2 2x18650, J3 U.FL-R-SMT_01_, J4 OMEGA2_HEADER, Q1 IRF7404, SW1 SW_POWER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

Commit message: finalize PCB
Connections:
- U2 pad 4: /SW_RST -> GND
