File: hardware/node/node.kicad_sch (KiCad schematic)
At the start: 61 parts, among them IC1 MCP73844-840I_MS, IC2 LM2576SX-3.3_NOPB, IC3 LM2585S-12_NOPB, IC4 NEO-M9N-00B, J1 USB4135-GF-A, J2 2x18650, J3 U.FL-R-SMT_01_, J4 OMEGA2_HEADER, Q1 IRF7404, SW1 SW_POWER, U1 ADS1115IDGS, U2 Omega2S

Commit message: PCB Layout
Parts:
- removed D3, D4: 550mV, symbol Device:D_Schottky
- removed J1: USB4135-GF-A, USB4135GFA, symbol USB4135-GF-A:USB4135-GF-A
- removed U1: ADS1115IDGS, Package_SO:TSSOP-10_3x3mm_P0.5mm, symbol Analog_ADC:ADS1115IDGS
- added D3: 550mV, B520C-13-F:DIOM7959X250N, symbol B520C-13-F:B520C-13-F
- added D4: 550mV, SS24FL:SODFL3617X108N, symbol SS24FL:SS24FL
- added D9: D_TVS, Diode_SMD:D_SOD-523, symbol Device:D_TVS
- added J1: USB4140-GF-0070-C, USB4140-GF-0070-C:USB4140GF0070C, symbol USB4140-GF-0070-C:USB4140-GF-0070-C
- added U1: ADS1113IDGS, Package_SO:TSSOP-10_3x3mm_P0.5mm, symbol Analog_ADC:ADS1113IDGS
- C1: footprint EEE1AA220WR -> EEE-FN1E100R:EEE1AA220WR
- C11: footprint (none) -> Capacitor_SMD:C_0402_1005Metric_Pad0.74x0.62mm_HandSolder
- C12, C6: footprint EEE1AA220WR -> KiCad:EEE1AA220WR
- C4, C5, C7: footprint CAPAE660X800N -> UUD1C221MCL1GS:CAPAE660X800N
- C8: footprint 16SVF180M -> 16SVPC100M:16SVF180M
- C9: footprint 16SVF1000M -> 16SVPF1000M:16SVF1000M
- D1, D2, D5, D7, D8: footprint (none) -> LED_SMD:LED_0805_2012Metric_Pad1.15x1.40mm_HandSolder
- D6: footprint Diode_THT:D_DO-41_SOD81_P10.16mm_Horizontal -> Diode_THT:D_A-405_P10.16mm_Horizontal
- F1: footprint (none) -> Fuse:Fuse_1206_3216Metric_Pad1.42x1.75mm_HandSolder
- H1, H2, H3, H4: footprint (none) -> MountingHole:MountingHole_3.2mm_M3
- IC1: footprint SOP65P490X110-8N -> MCP73844:SOP65P490X110-8N
- IC2: footprint KTT0005B -> LM2576SX-3.3_NOPB:KTT0005B
- IC3: footprint TO170P1435X465-6N -> LM2585S-12_NOPB:TO170P1435X465-6N
- IC4: footprint NEOM9N00B -> NEO-M9N-00B:NEOM9N00B
- J2: footprint 1123 -> 1123:1123
- J3: footprint UFLRSMT01 -> U.FL-R-SMT_01_:UFLRSMT01
- J4: footprint (none) -> Connector_PinSocket_2.00mm:PinSocket_1x06_P2.00mm_Vertical
- L1: footprint (none) -> 74437429203101:74437429203101
- L2: footprint (none) -> MSS1210-683MED:INDPM120120X1020N
- L3: footprint (none) -> Inductor_SMD:L_0603_1608Metric_Pad1.05x0.95mm_HandSolder
- R1, R10, R11, R12, R13, R14, R15, R17, R18, R19, R2, R20, R3, R5, R6, R7, R8, R9: footprint (none) -> Resistor_SMD:R_0603_1608Metric_Pad0.98x0.95mm_HandSolder
- R16: footprint (none) -> Resistor_SMD:R_1206_3216Metric_Pad1.30x1.75mm_HandSolder
- R4: footprint (none) -> Resistor_SMD:R_0805_2012Metric_Pad1.20x1.40mm_HandSolder
- SW1: footprint (none) -> L101011MS02Q:CKC5106-ND
Connections:
- net +12V: now also D4.1
- net +3.3V: now also U1.8 (VDD)
- net +5V: now also F1.1; no longer F1.2
- net GND: now also D3.2, D9.2 (A2), J1.A12 (GND_1), J1.B12 (GND_2), U1.1 (ADDR), U1.3 (GND)
- net GPS_ANT: now also D9.1 (A1)
- net I2C_SCL: now also U1.10 (SCL)
- net I2C_SDA: now also U1.9 (SDA)
- net at IC3.4 (SWITCH), L2.2: now also D4.2
- net at R1.2: now also J1.MH1, J1.MH2, J1.MH3, J1.MH4
- net at R3.1: now also J1.B5 (CC2)
- net at R6.1: now also J1.A5 (CC1)
- net at IC2.2 (OUTPUT), L1.1: now also D3.1
- net at R10.1, R9.2: now also U1.4 (AIN0)
- new net: F1.2, J1.A9 (VBUS_1), J1.B9 (VBUS_2)
Other:
- moved on the sheet: D1, R5

Commit message: finalize PCB
Parts:
- added C14: 0.1uF, Capacitor_SMD:C_1206_3216Metric_Pad1.33x1.80mm_HandSolder, symbol Device:C
- added R21: 50k, Resistor_SMD:R_0603_1608Metric_Pad0.98x0.95mm_HandSolder, symbol Device:R
Connections:
- net SW_RST is gone; now on net GND: U2.4 (SW_RST/GPIO_38)
- net +3.3V: now also C14.1, R21.1
- net GND: now also C14.2
- net at U2.5 (~{HW_RST}): now also R21.2
Changed lines of the file:
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@@
     (stroke (width 0) (type default) (color 0 0 0 0))
   )
+  (wire (pts (xy 275.59 58.42) (xy 271.78 58.42))
+    (stroke (width 0) (type default) (color 0 0 0 0))
+  )
   (wire (pts (xy 105.41 139.7) (xy 116.84 139.7))
     (stroke (width 0) (type default) (color 0 0 0 0))
@@
     (stroke (width 0) (type default) (color 0 0 0 0))
   )
+  (wire (pts (xy 275.59 54.61) (xy 275.59 58.42))
+    (stroke (width 0) (type default) (color 0 0 0 0))
+  )
   (wire (pts (xy 116.84 158.75) (xy 116.84 173.99))
     (stroke (width 0) (type default) (color 0 0 0 0))
@@
     (effects (font (size 1.27 1.27)) (justify right bottom))
   )
-  (label "SW_RST" (at 275.59 63.5 0)
-    (effects (font (size 1.27 1.27)) (justify left bottom))
-  )
   (label "VDD_FLASH" (at 246.38 44.45 0)
     (effects (font (size 1.27 1.27)) (justify left bottom))
@@
     (pin "1")
   )
+  (symbol (lib_id "Device:R") (at 275.59 50.8 0) (unit 1)
+    (in_bom yes) (on_board yes) (fields_autoplaced)
+    (property "Reference" "R21" (id 0) (at 278.13 49.5299 0)
+      (effects (font (size 1.27 1.27)) (justify left))
+    )
+    (property "Value" "50k" (id 1) (at 278.13 52.0699 0)
+      (effects (font (size 1.27 1.27)) (justify left))
+    )
+    (property "Footprint" "Resistor_SMD:R_0603_1608Metric_Pad0.98x0.95mm_HandSolder" (id 2) (at 273.812 50.8 90)
+      (effects (font (size 1.27 1.27)) hide)
+    )
+    (property "Datasheet" "~" (id 3) (at 275.59 50.8 0)
+      (effects (font (size 1.27 1.27)) hide)
+    )
+    (pin "1")
+    (pin "2")
+  )
   (symbol (lib_id "power:GND") (at 49.53 87.63 0) (unit 1)
     (in_bom yes) (on_board yes) (fields_autoplaced)
@@
     (pin "MH4")
   )
+  (symbol (lib_id "power:+3.3V") (at 275.59 46.99 0) (unit 1)
+    (in_bom yes) (on_board yes)
+    (property "Reference" "#PWR0109" (id 0) (at 275.59 50.8 0)
+      (effects (font (size 1.27 1.27)) hide)
+    )
+    (property "Value" "+3.3V" (id 1) (at 275.59 43.18 0))
+    (property "Footprint" "" (id 2) (at 275.59 46.99 0)
+      (effects (font (size 1.27 1.27)) hide)
+    )
+    (property "Datasheet" "" (id 3) (at 275.59 46.99 0)
+      (effects (font (size 1.27 1.27)) hide)
+    )
+    (pin "1")
+  )
   (symbol (lib_id "Device:R") (at 44.45 147.32 90) (unit 1)
     (in_bom yes) (on_board yes)
@@
     (pin "2")
   )
+  (symbol (lib_id "power:GND") (at 275.59 63.5 90) (unit 1)
+    (in_bom yes) (on_board yes) (fields_autoplaced)
+    (property "Reference" "#PWR?" (id 0) (at 281.94 63.5 0)
+      (effects (font (size 1.27 1.27)) hide)
+    )
+    (property "Value" "GND" (id 1) (at 279.4 63.4999 90)
+      (effects (font (size 1.27 1.27)) (justify right))
+    )
+    (property "Footprint" "" (id 2) (at 275.59 63.5 0)
+      (effects (font (size 1.27 1.27)) hide)
+    )
+    (property "Datasheet" "" (id 3) (at 275.59 63.5 0)
+      (effects (font (size 1.27 1.27)) hide)
+    )
+    (pin "1")
+  )
   (symbol (lib_id "EEE-FN1E100R:EEE-FN1E100R") (at 21.59 151.13 270) (unit 1)
     (in_bom yes) (on_board yes) (fields_autoplaced)
@@
     (pin "2")
   )
+  (symbol (lib_id "power:GND") (at 137.16 27.94 0) (unit 1)
+    (in_bom yes) (on_board yes) (fields_autoplaced)
+    (property "Reference" "#PWR0107" (id 0) (at 137.16 34.29 0)
+      (effects (font (size 1.27 1.27)) hide)
+    )
+    (property "Value" "GND" (id 1) (at 137.16 33.02 0))
+    (property "Footprint" "" (id 2) (at 137.16 27.94 0)
+      (effects (font (size 1.27 1.27)) hide)
+    )
+    (property "Datasheet" "" (id 3) (at 137.16 27.94 0)
+      (effects (font (size 1.27 1.27)) hide)
+    )
+    (pin "1")
+  )
   (symbol (lib_id "Device:LED") (at 172.72 71.12 0) (unit 1)
     (in_bom yes) (on_board yes)
@@
     (pin "2")
   )
+  (symbol (lib_id "power:+3.3V") (at 137.16 20.32 0) (unit 1)
+    (in_bom yes) (on_board yes)
+    (property "Reference" "#PWR0106" (id 0) (at 137.16 24.13 0)
+      (effects (font (size 1.27 1.27)) hide)
+    )
+    (property "Value" "+3.3V" (id 1) (at 137.16 16.51 0))
+    (property "Footprint" "" (id 2) (at 137.16 20.32 0)
+      (effects (font (size 1.27 1.27)) hide)
+    )
+    (property "Datasheet" "" (id 3) (at 137.16 20.32 0)
+      (effects (font (size 1.27 1.27)) hide)
+    )
+    (pin "1")
+  )
   (symbol (lib_id "power:GND") (at 140.97 68.58 0) (unit 1)
     (in_bom yes) (on_board yes) (fields_autoplaced)
@@
     (pin "1")
   )
+  (symbol (lib_id "Device:C") (at 137.16 24.13 0) (unit 1)
+    (in_bom yes) (on_board yes)
+    (property "Reference" "C14" (id 0) (at 139.7 22.86 0)
+      (effects (font (size 1.27 1.27)) (justify left))
+    )
+    (property "Value" "0.1uF" (id 1) (at 139.7 25.4 0)
+      (effects (font (size 1.27 1.27)) (justify left))
+    )
+    (property "Footprint" "Capacitor_SMD:C_1206_3216Metric_Pad1.33x1.80mm_HandSolder" (id 2) (at 138.1252 27.94 0)
+      (effects (font (size 1.27 1.27)) hide)
+    )
+    (property "Datasheet" "~" (id 3) (at 137.16 24.13 0)
+      (effects (font (size 1.27 1.27)) hide)
+    )
+    (pin "1")
+    (pin "2")
+  )
   (symbol (lib_id "16SVPC100M:16SVPC100M") (at 118.11 82.55 270) (unit 1)
     (in_bom yes) (on_board yes) (fields_autoplaced)
@@
       (reference "#PWR0105") (unit 1) (value "GND") (footprint "")
     )
+    (path "/b475ddc6-a3f8-42a3-9045-9138b9fe7c6e"
+      (reference "#PWR0106") (unit 1) (value "+3.3V") (footprint "")
+    )
+    (path "/9b5b86a9-c486-4e72-9dff-2f7b654f8685"
+      (reference "#PWR0107") (unit 1) (value "GND") (footprint "")
+    )
+    (path "/5385c658-699b-4152-8ec6-88c297b19a29"
+      (reference "#PWR0109") (unit 1) (value "+3.3V") (footprint "")
+    )
+    (path "/935b8990-f06d-4a90-ae14-1b7a209ea08b"
+      (reference "#PWR?") (unit 1) (value "GND") (footprint "")
+    )
     (path "/9518251b-a2a4-4f16-a0e5-e54284346937"
       (reference "C1") (unit 1) (value "10uF") (footprint "EEE-FN1E100R:EEE1AA220WR")
@@
       (reference "C13") (unit 1) (value "0.1uF") (footprint "Capacitor_SMD:C_1206_3216Metric_Pad1.33x1.80mm_HandSolder")
     )
+    (path "/c58a07a1-043a-4099-b165-3c63721e1e6a"
+      (reference "C14") (unit 1) (value "0.1uF") (footprint "Capacitor_SMD:C_1206_3216Metric_Pad1.33x1.80mm_HandSolder")
+    )
     (path "/a385e8d4-1558-4331-b3ba-3c8fefb4e262"
       (reference "D1") (unit 1) (value "LED_USB") (footprint "LED_SMD:LED_0805_2012Metric_Pad1.15x1.40mm_HandSolder")
@@
       (reference "R20") (unit 1) (value "22") (footprint "Resistor_SMD:R_0603_1608Metric_Pad0.98x0.95mm_HandSolder")
     )
+    (path "/18bee9c9-f427-4985-8854-6ac1bdd57903"
+      (reference "R21") (unit 1) (value "50k") (footprint "Resistor_SMD:R_0603_1608Metric_Pad0.98x0.95mm_HandSolder")
+    )
     (path "/8861aac9-d1da-4c05-9d0d-c33ec8cf5cdf"

Commit message: fix PCB dimensions to fit new case, remove USB series resistors from schematic
Parts:
- removed R17, R18: 27, Resistor_SMD:R_0603_1608Metric_Pad0.98x0.95mm_HandSolder, symbol Device:R
- removed R19, R20: 22, Resistor_SMD:R_0603_1608Metric_Pad0.98x0.95mm_HandSolder, symbol Device:R
Connections:
- net GPS_DM: now also IC4.5 (USB_DM), U2.62 (USB_DM)
- net GPS_DP: now also IC4.6 (USB_DP), U2.61 (USB_DP)
Changed lines of the file:
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@@
     (stroke (width 0) (type default) (color 0 0 0 0))
   )
-  (wire (pts (xy 204.47 162.56) (xy 204.47 158.75))
-    (stroke (width 0) (type default) (color 0 0 0 0))
-  )
   (wire (pts (xy 96.52 133.35) (xy 96.52 139.7))
     (stroke (width 0) (type default) (color 0 0 0 0))
@@
     (stroke (width 0) (type default) (color 0 0 0 0))
   )
-  (wire (pts (xy 208.28 162.56) (xy 208.28 158.75))
-    (stroke (width 0) (type default) (color 0 0 0 0))
-  )
   (wire (pts (xy 95.25 99.06) (xy 95.25 100.33))
     (stroke (width 0) (type default) (color 0 0 0 0))
@@
     (stroke (width 0) (type default) (color 0 0 0 0))
   )
-  (wire (pts (xy 200.66 69.85) (xy 200.66 66.04))
-    (stroke (width 0) (type default) (color 0 0 0 0))
-  )
   (wire (pts (xy 81.28 43.18) (xy 85.09 43.18))
     (stroke (width 0) (type default) (color 0 0 0 0))
@@
     (stroke (width 0) (type default) (color 0 0 0 0))
   )
-  (wire (pts (xy 204.47 69.85) (xy 204.47 66.04))
-    (stroke (width 0) (type default) (color 0 0 0 0))
-  )
   (wire (pts (xy 50.8 158.75) (xy 50.8 160.02))
     (stroke (width 0) (type default) (color 0 0 0 0))
@@
     (effects (font (size 1.27 1.27)) (justify right bottom))
   )
-  (label "GPS_DM" (at 204.47 162.56 180)
+  (label "GPS_DM" (at 204.47 151.13 180)
     (effects (font (size 1.27 1.27)) (justify right bottom))
   )
@@
     (effects (font (size 1.27 1.27)) (justify right bottom))
   )
-  (label "GPS_DM" (at 200.66 69.85 180)
+  (label "GPS_DM" (at 200.66 58.42 180)
     (effects (font (size 1.27 1.27)) (justify right bottom))
   )
@@
     (effects (font (size 1.27 1.27)) (justify left bottom))
   )
-  (label "GPS_DP" (at 208.28 162.56 0)
+  (label "GPS_DP" (at 208.28 151.13 0)
     (effects (font (size 1.27 1.27)) (justify left bottom))
   )
@@
     (effects (font (size 1.27 1.27)) (justify left bottom))
   )
-  (label "GPS_DP" (at 204.47 69.85 0)
+  (label "GPS_DP" (at 204.47 58.42 0)
     (effects (font (size 1.27 1.27)) (justify left bottom))
   )
@@
     )
   )
-  (symbol (lib_id "Device:R") (at 208.28 154.94 0) (unit 1)
-    (in_bom yes) (on_board yes)
-    (property "Reference" "R20" (id 0) (at 209.55 153.67 0)
-      (effects (font (size 1.27 1.27)) (justify left))
-    )
-    (property "Value" "22" (id 1) (at 209.55 156.21 0)
-      (effects (font (size 1.27 1.27)) (justify left))
-    )
-    (property "Footprint" "Resistor_SMD:R_0603_1608Metric_Pad0.98x0.95mm_HandSolder" (id 2) (at 206.502 154.94 90)
-      (effects (font (size 1.27 1.27)) hide)
-    )
-    (property "Datasheet" "~" (id 3) (at 208.28 154.94 0)
-      (effects (font (size 1.27 1.27)) hide)
-    )
-    (pin "1")
-    (pin "2")
-  )
   (symbol (lib_id "power:GND") (at 232.41 44.45 0) (unit 1)
     (in_bom yes) (on_board yes)
@@
     (pin "2")
   )
-  (symbol (lib_id "Device:R") (at 200.66 62.23 0) (unit 1)
-    (in_bom yes) (on_board yes)
-    (property "Reference" "R17" (id 0) (at 195.58 60.96 0)
-      (effects (font (size 1.27 1.27)) (justify left))
-    )
-    (property "Value" "27" (id 1) (at 196.85 63.5 0)
-      (effects (font (size 1.27 1.27)) (justify left))
-    )
-    (property "Footprint" "Resistor_SMD:R_0603_1608Metric_Pad0.98x0.95mm_HandSolder" (id 2) (at 198.882 62.23 90)
-      (effects (font (size 1.27 1.27)) hide)
-    )
-    (property "Datasheet" "~" (id 3) (at 200.66 62.23 0)
-      (effects (font (size 1.27 1.27)) hide)
-    )
-    (pin "1")
-    (pin "2")
-  )
   (symbol (lib_id "power:GND") (at 208.28 49.53 0) (unit 1)
     (in_bom yes) (on_board yes) (fields_autoplaced)
@@
     (pin "2")
   )
-  (symbol (lib_id "Device:R") (at 204.47 62.23 0) (unit 1)
-    (in_bom yes) (on_board yes)
-    (property "Reference" "R18" (id 0) (at 205.74 60.96 0)
-      (effects (font (size 1.27 1.27)) (justify left))
-    )
-    (property "Value" "27" (id 1) (at 205.74 63.5 0)
-      (effects (font (size 1.27 1.27)) (justify left))
-    )
-    (property "Footprint" "Resistor_SMD:R_0603_1608Metric_Pad0.98x0.95mm_HandSolder" (id 2) (at 202.692 62.23 90)
-      (effects (font (size 1.27 1.27)) hide)
-    )
-    (property "Datasheet" "~" (id 3) (at 204.47 62.23 0)
-      (effects (font (size 1.27 1.27)) hide)
-    )
-    (pin "1")
-    (pin "2")
-  )
   (symbol (lib_id "UUD1C221MCL1GS:UUD1C221MCL1GS") (at 99.06 100.33 270) (unit 1)
     (in_bom yes) (on_board yes)
@@
     (pin "2")
   )
-  (symbol (lib_id "Device:R") (at 204.47 154.94 0) (unit 1)
-    (in_bom yes) (on_board yes)
-    (property "Reference" "R19" (id 0) (at 199.39 153.67 0)
-      (effects (font (size 1.27 1.27)) (justify left))
-    )
-    (property "Value" "22" (id 1) (at 200.66 156.21 0)
-      (effects (font (size 1.27 1.27)) (justify left))
-    )
-    (property "Footprint" "Resistor_SMD:R_0603_1608Metric_Pad0.98x0.95mm_HandSolder" (id 2) (at 202.692 154.94 90)
-      (effects (font (size 1.27 1.27)) hide)
-    )
-    (property "Datasheet" "~" (id 3) (at 204.47 154.94 0)
-      (effects (font (size 1.27 1.27)) hide)
-    )
-    (pin "1")
-    (pin "2")
-  )
   (symbol (lib_id "Device:R") (at 38.1 76.2 0) (unit 1)
     (in_bom yes) (on_board yes)
@@
       (reference "R16") (unit 1) (value "10") (footprint "Resistor_SMD:R_1206_3216Metric_Pad1.30x1.75mm_HandSolder")
     )
-    (path "/4f278437-ab73-4697-9129-e426793306ea"
-      (reference "R17") (unit 1) (value "27") (footprint "Resistor_SMD:R_0603_1608Metric_Pad0.98x0.95mm_HandSolder")
-    )
-    (path "/9e6f02f9-429a-4d23-9a10-458bbaf21675"
-      (reference "R18") (unit 1) (value "27") (footprint "Resistor_SMD:R_0603_1608Metric_Pad0.98x0.95mm_HandSolder")
-    )
-    (path "/e0d220d5-33cf-4060-a6b0-a34163202010"
-      (reference "R19") (unit 1) (value "22") (footprint "Resistor_SMD:R_0603_1608Metric_Pad0.98x0.95mm_HandSolder")
-    )
-    (path "/13e70e84-ea1d-475f-837d-595d82b171e4"
-      (reference "R20") (unit 1) (value "22") (footprint "Resistor_SMD:R_0603_1608Metric_Pad0.98x0.95mm_HandSolder")
-    )
     (path "/18bee9c9-f427-4985-8854-6ac1bdd57903"
