File: hardware/node/node.kicad_pcb (KiCad board)
At the start: 2 copper layers, 168.9 x 109.2 mm, 64 parts, among them IC1 MCP73844-840I_MS, IC2 LM2576SX-3.3_NOPB, IC3 LM2585S-12_NOPB, IC4 NEO-M9N-00B, J1 USB4140-GF-0070-C, J2 2x18650, J3 U.FL-R-SMT_01_, J4 OMEGA2_HEADER, Q1 IRF7404, SW1 SW_POWER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

Commit message: fix PCB dimensions to fit new case, remove USB series resistors from schematic
Parts:
- moved H2 50.9 mm to (252.3, 20.3)
- moved H4 40.9 mm to (252.3, 156.2)
- moved H1 30.5 mm to (50.8, 20.3)
- moved H3 3.66 mm to (50.8, 156.2)
Connections:
- U2 pad 4: /SW_RST -> GND
Other:
- board size 168.9 x 109.2 mm -> 209.1 x 143.5 mm
- board text added: "CHeap Accessible Resilient Mesh v1.1"
- board text removed: "CHeap Accessible Resilient Mesh v1.0"

Commit message: push latest PCB
Parts:
- removed R17, R18: 27, Resistor_SMD:R_0603_1608Metric_Pad0.98x0.95mm_HandSolder
- removed R19, R20: 22, Resistor_SMD:R_0603_1608Metric_Pad0.98x0.95mm_HandSolder
- moved R11 25.2 mm to (155.4, 138.3)
- moved C14 25.2 mm to (209.0, 95.2)
- moved D8 25.2 mm to (182.0, 93.9)
- moved D9 25.2 mm to (188.1, 114.5)
- moved R14 25.2 mm to (141.0, 120.9)
- moved R15 25.2 mm to (141.0, 125.2)
- moved U2 25.2 mm to (162.1, 113.8)
- moved C12 25.2 mm to (141.3, 109.4)
- moved C13 25.2 mm to (148.5, 108.9)
- moved C3 25.2 mm to (132.5, 76.6)
- moved C6 25.2 mm to (140.3, 72.1)
- moved C7 25.2 mm to (111.0, 54.4)
- moved C8 25.2 mm to (82.3, 114.3)
- moved C9 25.2 mm to (111.8, 67.0)
- moved D2 25.2 mm to (122.6, 70.2)
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Connections:
- IC4 pad 5: Net-(IC4-Pad5) -> /GPS_DM
- IC4 pad 6: Net-(IC4-Pad6) -> /GPS_DP
- U2 pad 61: Net-(R20-Pad1) -> /GPS_DP
- U2 pad 62: Net-(R19-Pad1) -> /GPS_DM
Routing:
- net /GPS_DM: track 7.60 -> 21.9 mm
- net /GPS_DP: track 7.65 -> 21.9 mm
- net Net-(R19-Pad1): track 5.53 -> 0.00 mm
- net Net-(R20-Pad1): track 5.52 -> 0.00 mm
- net Net-(IC4-Pad6): track 5.24 -> 0.00 mm
- net Net-(IC4-Pad5): track 5.22 -> 0.00 mm
- net Net-(C6-Pad1): track 45.4 -> 47.1 mm
- net /VBAT: track 91.7 -> 92.9 mm
- net GND: vias 68 -> 79
- added copper zone on F.Cu, net Net-(C6-Pad1)
Other:
- outline, holes or cut-outs redrawn
- board text added: "BobaFET"
- board text added: "JLCJLCJLCJLC"
